File: VW-MTC1/Hardware/KiCad/MCU.kicad_sch (KiCad schematic)
At the start: 37 parts, among them J5 OLED, J6 QWIIC, J7 microSD, SW2 RESET, SW3 BOOT/MODE, SW4 START, U12 ISM330DHCX, U5 ESP32-S3-WROOM-1-N8R2

Commit message: Apply Rev B touch circuit, routed PCB and topology-tested BOM
Connections:
- net TOUCH_FINISH renamed TOUCH_BUSY
- net TOUCH_START renamed TOUCH_CS
- net TOUCH_WIRE renamed TOUCH_EXC
Changed lines of the file:
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@@
 	(title_block
 		(title "MCU: ESP32-S3, UI, IMU, storage, expansion")
-		(date "2026-10-19")
-		(rev "A")
+		(date "2026-10-21")
+		(rev "B")
 		(company "Voltwyn")
 		(comment 1 "VW-MTC1 MazeTrack Controller - MCU")
@@
 		)
 	)
-	(global_label "TOUCH_FINISH"
+	(global_label "TOUCH_BUSY"
 		(shape passive)
 		(at 74.93 64.77 0)
@@
 		)
 	)
-	(global_label "TOUCH_WIRE"
+	(global_label "TOUCH_EXC"
 		(shape passive)
 		(at 74.93 82.55 0)
@@
 		)
 	)
-	(global_label "TOUCH_START"
+	(global_label "TOUCH_CS"
 		(shape passive)
 		(at 74.93 85.09 0)
