File: VW-MTC1/Hardware/KiCad/Sensing.kicad_sch (KiCad schematic)
At the start: 45 parts, among them J3 HANDLE, Q2 AO3401A, Q3 AO3400A, U6 MCP6004-I/SL, U7 MCP3204-C/SL, U8 TPD4E05U06, U9 PRTR5V0U2X

Commit message: Apply Rev B touch circuit, routed PCB and topology-tested BOM
Parts:
- U7: symbol Analog_ADC:MCP3204 -> Voltwyn:MCP3204
Changed lines of the file:
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@@
 	(title_block
 		(title "Sensing: Hall front end, 12-bit ADC, handle I/O, haptics")
-		(date "2026-10-19")
-		(rev "A")
+		(date "2026-10-21")
+		(rev "B")
 		(company "Voltwyn")
 		(comment 1 "VW-MTC1 MazeTrack Controller - Sensing")
@@
 	)
 	(symbol
-		(lib_id "Analog_ADC:MCP3204")
+		(lib_id "Voltwyn:MCP3204")
 		(at 162.56 105.41 0)
 		(unit 1)
