File: VW-MTC1/Hardware/KiCad/VW-MTC1.kicad_pcb (KiCad board)
At the start: 4 copper layers, 90 x 60 mm, 154 parts, among them J1 USB-C, J2 BATT 1S, J3 HANDLE, J4 MAZE, J5 OLED, J6 QWIIC, J7 microSD, Q1 AO3401A, Q2 AO3401A, Q3 AO3400A, Q4 AO3400A, SW1 POWER, SW2 RESET, SW3 BOOT/MODE, SW4 START, U1 USBLC6-2SC6, U10 TPD4E05U06, U11 74LVC3G17, U12 ISM330DHCX, U3 LTC4054ES5-4.2, U4 LTC3536EMSE, U5 ESP32-S3-WROOM-1-N8R2, U6 MCP6004-I/SL, U7 MCP3204-C/SL, U8 TPD4E05U06, U9 PRTR5V0U2X

Commit message: Apply Rev B touch circuit, routed PCB and topology-tested BOM
Parts:
- added C40: 270pF C0G, Capacitor_SMD:C_0603_1608Metric, F.Cu at (181.5, 131.5)
- added C41: 100nF, Capacitor_SMD:C_0603_1608Metric, F.Cu at (151.8, 132.2)
- added C42: 100nF, Capacitor_SMD:C_0603_1608Metric, F.Cu at (151.8, 136.2)
- added C43: 4.7uF, Capacitor_SMD:C_0603_1608Metric, F.Cu at (151.8, 128.2)
- added C44: 1uF, Capacitor_SMD:C_0603_1608Metric, F.Cu at (151.8, 130.2)
- added C45: 1uF, Capacitor_SMD:C_0603_1608Metric, F.Cu at (163.2, 143.5)
- added C46: 1uF, Capacitor_SMD:C_0603_1608Metric, F.Cu at (161.5, 143.2)
- added R61: 187k 0.05%, Resistor_SMD:R_0603_1608Metric, F.Cu at (169.5, 136.0)
- added R62: 200k 0.05%, Resistor_SMD:R_0603_1608Metric, F.Cu at (171.5, 136.0)
- added R63: 187k 0.05%, Resistor_SMD:R_0603_1608Metric, F.Cu at (169.5, 145.6)
- added R64: 200k 0.05%, Resistor_SMD:R_0603_1608Metric, F.Cu at (171.5, 145.6)
- added R65: 187k 0.05%, Resistor_SMD:R_0603_1608Metric, F.Cu at (173.5, 136.0)
- added R66: 200k 0.05%, Resistor_SMD:R_0603_1608Metric, F.Cu at (175.5, 136.0)
- added R67: 100k 0.05%, Resistor_SMD:R_0603_1608Metric, F.Cu at (175.5, 131.5)
- added R68: 187k 0.05%, Resistor_SMD:R_0603_1608Metric, F.Cu at (177.5, 131.5)
- added R69: 200k 0.05%, Resistor_SMD:R_0603_1608Metric, F.Cu at (179.5, 131.5)
- added R70: 220R 0.05%, Resistor_SMD:R_0603_1608Metric, F.Cu at (160.0, 140.2)
- added R71: 100R 0.05%, Resistor_SMD:R_0603_1608Metric, F.Cu at (160.0, 138.5)
- added R72: 10k, Resistor_SMD:R_0603_1608Metric, F.Cu at (156.5, 140.2)
- added R73: 10k, Resistor_SMD:R_0603_1608Metric, F.Cu at (164.2, 127.8)
- added R74: 10R, Resistor_SMD:R_0603_1608Metric, F.Cu at (151.8, 134.2)
- added TP10: TOUCH_DRIVE, TestPoint:TestPoint_Pad_D1.5mm, B.Cu at (155.8, 137.5)
- added U13: ADS8344NB, Package_SO:SSOP-20_5.3x7.2mm_P0.65mm, F.Cu at (159.0, 133.2)
- added U14: REF3325, Package_TO_SOT_SMD:SOT-23, F.Cu at (158.5, 143.8)
- C34, C35, C36: value 27nF -> 270pF C0G
- R51, R53, R55: value 10k -> 1.15M
- R52, R54, R56: value 360k -> 100k 0.05%
- TP9: value TOUCH_WIRE -> TOUCH_EXC; moved to B.Cu
- U11: value 74LVC3G17 -> OPA4323; footprint Package_SO:VSSOP-8_2.3x2mm_P0.5mm -> Package_SO:TSSOP-14_4.4x5mm_P0.65mm
- moved R55 11.2 mm to (177.2, 139.5), turned to 180 degrees
- moved R56 11.0 mm to (175.5, 145.9)
- moved R51 9.65 mm to (177.2, 143.5), turned to 180 degrees
- moved C34 9.01 mm to (165.5, 136.0), turned to 90 degrees
- moved C37 8.96 mm to (163.2, 140.0), turned to 90 degrees
- moved C35 8.90 mm to (165.5, 145.6), turned to 90 degrees
- moved R54 8.68 mm to (167.5, 145.6), turned to 90 degrees
- moved R52 5.25 mm to (167.5, 136.0)
- moved U10 3.40 mm to (174.2, 139.5)
- moved C36 3.00 mm to (173.5, 145.6), turned to 90 degrees
- moved R53 2.76 mm to (177.2, 141.5), turned to 180 degrees
- moved U11 2.50 mm to (168.5, 141.0)
- turned TP9 to 180 degrees
Connections:
- R52 pad 1: +3V3 -> TOUCH_DRIVE
- R54 pad 1: +3V3 -> TOUCH_DRIVE
- R56 pad 1: +3V3 -> TOUCH_DRIVE
- TP9 pad 1: TOUCH_WIRE -> TOUCH_EXC
- U10 pad 1: MAZE_WIRE -> TCH_WIRE
- U10 pad 2: MAZE_START -> TCH_START
- U10 pad 4: MAZE_FINISH -> TCH_FIN
- U11 pad 1: TCH_WIRE -> TCH_ADC0
- U11 pad 2: TOUCH_START -> TCH_ADC0
- U11 pad 3: TCH_FIN -> TCH_WIRE
- U11 pad 4: GND -> +3V3
- U11 pad 5: TOUCH_FINISH -> TCH_START
- U11 pad 6: TCH_START -> TCH_ADC1
- U11 pad 7: TOUCH_WIRE -> TCH_ADC1
- U11 pad 8: +3V3 -> TCH_ADC2
- U5 pad 23: TOUCH_FINISH -> TOUCH_BUSY
- U5 pad 34: TOUCH_WIRE -> TOUCH_EXC
- U5 pad 35: TOUCH_START -> TOUCH_CS
Routing:
- net GND: track 116.2 -> 874.2 mm, vias 173 -> 153
- net +3V3: track 41.7 -> 346.3 mm, vias 41 -> 45
- net TOUCH_CS: track 0.00 -> 103.7 mm, vias 0 -> 2
- net TOUCH_EXC: track 0.00 -> 94.2 mm, vias 0 -> 3
- net TOUCH_START: track 89.9 -> 0.00 mm, vias 2 -> 0
- net TOUCH_WIRE: track 82.0 -> 0.00 mm, vias 2 -> 0
- net TOUCH_FINISH: track 69.0 -> 0.00 mm, vias 2 -> 0
- net TOUCH_DRIVE: track 0.00 -> 56.7 mm, vias 0 -> 3
- net +3V3_TOUCH: track 0.00 -> 51.9 mm
- net TOUCH_BUSY: track 0.00 -> 51.2 mm, vias 0 -> 2
- net MAZE_FINISH: track 30.7 -> 3.38 mm
- net MAZE_WIRE: track 26.5 -> 3.38 mm
- net +2V5_TOUCH: track 0.00 -> 22.4 mm, vias 0 -> 3
- net TCH_WIRE: track 7.88 -> 29.7 mm, vias 0 -> 2
- net TCH_REF: track 0.00 -> 18.5 mm, vias 0 -> 2
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